Commit message: Refactor URDF files for camera frames and joints

File: urdf/astra2.urdf.xacro (robot description, xacro)
@@ -4,5 +4,5 @@
      For more information, please see http://wiki.ros.org/sw_urdf_exporter -->
 <robot xmlns:xacro="http://ros.org/wiki/xacro" name="astra2">
-    <xacro:property name="mesh_path" value="package://orbbec_camera/meshes/astra2/" />
+    <xacro:property name="mesh_path" value="package://orbbec_description/meshes/astra2/" />
   <link
     name="camera_link">
@@ -23,5 +23,5 @@
     <visual>
       <origin
-        xyz="0 0 0"
+        xyz="-0.012323995999904 -0.0374999999985815 -0.0281503197112"
         rpy="0 0 0" />
       <geometry>
@@ -89,5 +89,5 @@
     type="fixed">
     <origin
-      xyz="0 0 0"
+      xyz="-0.012323995999904 -0.0374999999985815 -0.0281503197112"
       rpy="0 0 0" />
     <parent
@@ -99,5 +99,5 @@
   </joint>
   <link
-    name="camera_infra1_frame">
+    name="camera_ir_frame">
     <inertial>
       <origin
@@ -139,18 +139,18 @@
   </link>
   <joint
-    name="camera_infra1_frame"
-    type="fixed">
-    <origin
-      xyz="0.012323995999904 0.0374999999985815 0.0281503197112"
+    name="camera_ir_frame"
+    type="fixed">
+    <origin
+      xyz="0 0 0"
       rpy="0 0 0" />
     <parent
-      link="camera_bottom_screw_frame" />
-    <child
-      link="camera_infra1_frame" />
-    <axis
-      xyz="0 0 0" />
-  </joint>
-  <link
-    name="camera_infra1_optical_frame">
+      link="camera_depth_frame" />
+    <child
+      link="camera_ir_frame" />
+    <axis
+      xyz="0 0 0" />
+  </joint>
+  <link
+    name="camera_ir_optical_frame">
     <inertial>
       <origin
@@ -192,5 +192,5 @@
   </link>
   <joint
-    name="camera_infra1_optical_frame"
+    name="camera_ir_optical_frame"
     type="fixed">
     <origin
@@ -198,12 +198,12 @@
       rpy="-1.5707963267949 0 -1.5707963267949" />
     <parent
-      link="camera_infra1_frame" />
-    <child
-      link="camera_infra1_optical_frame" />
-    <axis
-      xyz="0 0 0" />
-  </joint>
-  <link
-    name="camera_colorl_frame">
+      link="camera_ir_frame" />
+    <child
+      link="camera_ir_optical_frame" />
+    <axis
+      xyz="0 0 0" />
+  </joint>
+  <link
+    name="camera_color_frame">
     <inertial>
       <origin
@@ -248,10 +248,10 @@
     type="fixed">
     <origin
-      xyz="0.014865995999904 0.0189999999985815 0.0281503197112"
+      xyz="0.0025420000310987234 -0.01850000023841858 0"
       rpy="0 0 0" />
     <parent
-      link="camera_bottom_screw_frame" />
-    <child
-      link="camera_colorl_frame" />
+      link="camera_depth_frame" />
+    <child
+      link="camera_color_frame" />
     <axis
       xyz="0 0 0" />
@@ -304,5 +304,5 @@
       rpy="-1.5707963267949 0 -1.5707963267949" />
     <parent
-      link="camera_colorl_frame" />
+      link="camera_color_frame" />
     <child
       link="camera_color_optical_frame" />
@@ -354,8 +354,8 @@
     type="fixed">
     <origin
-      xyz="0.012323995999904 0.0374999999985815 0.0281503197112"
+      xyz="0 0 0"
       rpy="0 0 0" />
     <parent
-      link="camera_bottom_screw_frame" />
+      link="camera_link" />
     <child
       link="camera_depth_frame" />

File: urdf/gemini2.urdf.xacro (robot description, xacro)
@@ -4,5 +4,5 @@
      For more information, please see http://wiki.ros.org/sw_urdf_exporter -->
 <robot xmlns:xacro="http://ros.org/wiki/xacro" name="gemini2">
-    <xacro:property name="mesh_path" value="package://orbbec_camera/meshes/gemini2/" />
+    <xacro:property name="mesh_path" value="package://orbbec_description/meshes/gemini2/" />
   <link
     name="camera_link">
@@ -23,5 +23,5 @@
     <visual>
       <origin
-        xyz="0 0 0"
+        xyz="-0.01491 -0.025 -0.0125"
         rpy="0 0 0" />
       <geometry>
@@ -89,5 +89,5 @@
     type="fixed">
     <origin
-      xyz="0 0 0"
+      xyz="-0.01491 -0.025 -0.0125"
       rpy="0 0 0" />
     <parent
@@ -99,5 +99,5 @@
   </joint>
   <link
-    name="camera_infra1_frame">
+    name="camera_right_ir_frame">
     <inertial>
       <origin
@@ -139,18 +139,18 @@
   </link>
   <joint
-    name="camera_infra1_frame"
-    type="fixed">
-    <origin
-      xyz="0.01491 -0.025 0.0125"
+    name="camera_right_ir_frame"
+    type="fixed">
+    <origin
+      xyz="0 -0.05000000074505806 0"
       rpy="0 0 0" />
     <parent
-      link="camera_botter_screw_frame" />
-    <child
-      link="camera_infra1_frame" />
-    <axis
-      xyz="0 0 0" />
-  </joint>
-  <link
-    name="camera_infra1_optical_frame">
+      link="camera_depth_frame" />
+    <child
+      link="camera_right_ir_frame" />
+    <axis
+      xyz="0 0 0" />
+  </joint>
+  <link
+    name="camera_right_ir_optical_frame">
     <inertial>
       <origin
@@ -192,5 +192,5 @@
   </link>
   <joint
-    name="camera_infra1_optical_frame"
+    name="camera_right_ir_optical_frame"
     type="fixed">
     <origin
@@ -198,7 +198,7 @@
       rpy="-1.5707963267949 0 -1.5707963267949" />
     <parent
-      link="camera_infra1_frame" />
-    <child
-      link="camera_infra1_optical_frame" />
+      link="camera_right_ir_frame" />
+    <child
+      link="camera_right_ir_optical_frame" />
     <axis
       xyz="0 0 0" />
@@ -248,8 +248,8 @@
     type="fixed">
     <origin
-      xyz="0.01682 0.010995 0.012505"
-      rpy="-1.5707963267949 0 -1.5707963267949" />
-    <parent
-      link="camera_botter_screw_frame" />
+      xyz="0.0019099999917671084 -0.01400499977171421 4.999999873689376e-06"
+      rpy="0 0 0" />
+    <parent
+      link="camera_depth_frame" />
     <child
       link="camera_color_frame" />
@@ -302,5 +302,5 @@
     <origin
       xyz="0 0 0"
-      rpy="0 0 0" />
+      rpy="-1.5707963267949 0 -1.5707963267949" />
     <parent
       link="camera_color_frame" />
@@ -311,5 +311,5 @@
   </joint>
   <link
-    name="camera_infra2_frame">
+    name="camera_left_ir_frame">
     <inertial>
       <origin
@@ -351,18 +351,18 @@
   </link>
   <joint
-    name="camera_infra2_frame"
-    type="fixed">
-    <origin
-      xyz="0.01491 0.025 0.0125"
+    name="camera_left_ir_frame"
+    type="fixed">
+    <origin
+      xyz="0 0 0"
       rpy="0 0 0" />
     <parent
-      link="camera_botter_screw_frame" />
-    <child
-      link="camera_infra2_frame" />
-    <axis
-      xyz="0 0 0" />
-  </joint>
-  <link
-    name="camera_infra2_optical_frame">
+      link="camera_link" />
+    <child
+      link="camera_left_ir_frame" />
+    <axis
+      xyz="0 0 0" />
+  </joint>
+  <link
+    name="camera_left_ir_optical_frame">
     <inertial>
       <origin
@@ -404,5 +404,5 @@
   </link>
   <joint
-    name="camera_infra2_optical_frame"
+    name="camera_left_ir_optical_frame"
     type="fixed">
     <origin
@@ -410,7 +410,7 @@
       rpy="-1.5707963267949 0 -1.5707963267949" />
     <parent
-      link="camera_infra2_frame" />
-    <child
-      link="camera_infra2_optical_frame" />
+      link="camera_left_ir_frame" />
+    <child
+      link="camera_left_ir_optical_frame" />
     <axis
       xyz="0 0 0" />
@@ -460,8 +460,8 @@
     type="fixed">
     <origin
-      xyz="0.01491 0.025 0.0125"
+      xyz="0 0 0"
       rpy="0 0 0" />
     <parent
-      link="camera_botter_screw_frame" />
+      link="camera_link" />
     <child
       link="camera_depth_frame" />

File: urdf/gemini2L.urdf.xacro (robot description, xacro)
@@ -4,5 +4,5 @@
      For more information, please see http://wiki.ros.org/sw_urdf_exporter -->
 <robot xmlns:xacro="http://ros.org/wiki/xacro" name="gemini2l">
-    <xacro:property name="mesh_path" value="package://orbbec_camera/meshes/gemini2l/" />
+    <xacro:property name="mesh_path" value="package://orbbec_description/meshes/gemini2l/" />
   <link
     name="camera_link">
@@ -23,5 +23,5 @@
     <visual>
       <origin
-        xyz="0 0 0"
+        xyz="-0.01033 -0.05 -0.0145"
         rpy="0 0 0" />
       <geometry>
@@ -89,5 +89,5 @@
     type="fixed">
     <origin
-      xyz="0 0 0"
+      xyz="-0.01033 -0.05 -0.0145"
       rpy="0 0 0" />
     <parent
@@ -99,5 +99,5 @@
   </joint>
   <link
-    name="camera_IR2_frame">
+    name="camera_right_ir_frame">
     <inertial>
       <origin
@@ -139,18 +139,18 @@
   </link>
   <joint
-    name="camera_IR2_frame"
-    type="fixed">
-    <origin
-      xyz="0.01033 -0.05 0.0145"
+    name="camera_right_ir_frame"
+    type="fixed">
+    <origin
+      xyz="0 -0.1 0"
       rpy="0 0 0" />
     <parent
-      link="camera_bottom_screw_frame" />
-    <child
-      link="camera_IR2_frame" />
-    <axis
-      xyz="0 0 0" />
-  </joint>
-  <link
-    name="camera_IR2_optical_frame">
+      link="camera_depth_frame" />
+    <child
+      link="camera_right_ir_frame" />
+    <axis
+      xyz="0 0 0" />
+  </joint>
+  <link
+    name="camera_right_ir_optical_frame">
     <inertial>
       <origin
@@ -192,5 +192,5 @@
   </link>
   <joint
-    name="camera_IR2_optical_frame"
+    name="camera_right_ir_optical_frame"
     type="fixed">
     <origin
@@ -198,12 +198,12 @@
       rpy="-1.5708 0 -1.5708" />
     <parent
-      link="camera_IR2_frame" />
-    <child
-      link="camera_IR2_optical_frame" />
-    <axis
-      xyz="0 0 0" />
-  </joint>
-  <link
-    name="camera_IR1_frame">
+      link="camera_right_ir_frame" />
+    <child
+      link="camera_right_ir_optical_frame" />
+    <axis
+      xyz="0 0 0" />
+  </joint>
+  <link
+    name="camera_left_ir_frame">
     <inertial>
       <origin
@@ -245,18 +245,18 @@
   </link>
   <joint
-    name="camera_IR1_frame"
-    type="fixed">
-    <origin
-      xyz="0.01033 0.05 0.0145"
+    name="camera_left_ir_frame"
+    type="fixed">
+    <origin
+      xyz="0 0 0"
       rpy="0 0 0" />
     <parent
-      link="camera_bottom_screw_frame" />
-    <child
-      link="camera_IR1_frame" />
-    <axis
-      xyz="0 0 0" />
-  </joint>
-  <link
-    name="camera_IR1_optical_frame">
+      link="camera_depth_frame" />
+    <child
+      link="camera_left_ir_frame" />
+    <axis
+      xyz="0 0 0" />
+  </joint>
+  <link
+    name="camera_left_ir_optical_frame">
     <inertial>
       <origin
@@ -298,5 +298,5 @@
   </link>
   <joint
-    name="camera_IR1_optical_frame"
+    name="camera_left_ir_optical_frame"
     type="fixed">
     <origin
@@ -304,7 +304,7 @@
       rpy="-1.5708 0 -1.5708" />
     <parent
-      link="camera_IR1_frame" />
-    <child
-      link="camera_IR1_optical_frame" />
+      link="camera_left_ir_frame" />
+    <child
+      link="camera_left_ir_optical_frame" />
     <axis
       xyz="0 0 0" />
@@ -354,8 +354,8 @@
     type="fixed">
     <origin
-      xyz="0.010330000039789 0.025 0.0145"
+      xyz="3.9789e-11 -0.025 0"
       rpy="0 0 0" />
     <parent
-      link="camera_bottom_screw_frame" />
+      link="camera_depth_frame" />
     <child
       link="camera_color_frame" />
@@ -364,5 +364,5 @@
   </joint>
   <link
-    name="camera_rgb_optical_frame">
+    name="camera_color_optical_frame">
     <inertial>
       <origin
@@ -404,5 +404,5 @@
   </link>
   <joint
-    name="camera_rgb_optical_frame"
+    name="camera_color_optical_frame"
     type="fixed">
     <origin
@@ -412,5 +412,5 @@
       link="camera_color_frame" />
     <child
-      link="camera_rgb_optical_frame" />
+      link="camera_color_optical_frame" />
     <axis
       xyz="0 0 0" />
@@ -460,8 +460,8 @@
     type="fixed">
     <origin
-      xyz="-0.00473999996021007 0.034841019999999 0.017079659999999"
+      xyz="-0.01507 -0.015159 0.0025797"
       rpy="0 0 0" />
     <parent
-      link="camera_bottom_screw_frame" />
+      link="camera_depth_frame" />
     <child
       link="camera_imu_frame" />
@@ -513,8 +513,8 @@
     type="fixed">
     <origin
-      xyz="0.010330000039789 0.05 0.0145"
+      xyz="0 0 0"
       rpy="0 0 0" />
     <parent
-      link="camera_bottom_screw_frame" />
+      link="camera_link" />
     <child
       link="camera_depth_frame" />

File: urdf/gemini335L_336L.urdf.xacro (robot description, xacro)
@@ -4,5 +4,5 @@
      For more information, please see http://wiki.ros.org/sw_urdf_exporter -->
 <robot xmlns:xacro="http://ros.org/wiki/xacro" name="gemini_335L_336L">
-    <xacro:property name="mesh_path" value="package://orbbec_camera/meshes/gemini335L_336L/" />
+    <xacro:property name="mesh_path" value="package://orbbec_description/meshes/gemini335L_336L/" />
   <link
     name="camera_link">
@@ -23,5 +23,5 @@
     <visual>
       <origin
-        xyz="0 0 0"
+        xyz="-0.011715 -0.0475 -0.014311"
         rpy="0 0 0" />
       <geometry>
@@ -89,5 +89,5 @@
     type="fixed">
     <origin
-      xyz="0 0 0"
+      xyz="-0.011715 -0.0475 -0.014311"
       rpy="0 0 0" />
     <parent
@@ -142,8 +142,8 @@
     type="fixed">
     <origin
-      xyz="-0.002535 0.039634 0.013243"
+      xyz="-0.01425 -0.007866 -0.001068"
       rpy="0 0 0" />
     <parent
-      link="camera_color_screw_frame" />
+      link="camera_depth_frame" />
     <child
       link="camera_IMU_frame" />
@@ -195,8 +195,8 @@
     type="fixed">
     <origin
-      xyz="0.011715 0.0475 0.014311"
+      xyz="0 0 0"
       rpy="0 0 0" />
     <parent
-      link="camera_color_screw_frame" />
+      link="camera_link" />
     <child
       link="camera_depth_frame" />
@@ -205,5 +205,5 @@
   </joint>
   <link
-    name="camera_infra1_frame">
+    name="camera_left_ir_frame">
     <inertial>
       <origin
@@ -245,18 +245,18 @@
   </link>
   <joint
-    name="camera_infra1_frame"
-    type="fixed">
-    <origin
-      xyz="0.011715 0.0475 0.014311"
+    name="camera_left_ir_frame"
+    type="fixed">
+    <origin
+      xyz="0 0 0"
       rpy="0 0 0" />
     <parent
-      link="camera_color_screw_frame" />
-    <child
-      link="camera_infra1_frame" />
-    <axis
-      xyz="0 0 0" />
-  </joint>
-  <link
-    name="camera_infra1_optical_frame">
+      link="camera_depth_frame" />
+    <child
+      link="camera_left_ir_frame" />
+    <axis
+      xyz="0 0 0" />
+  </joint>
+  <link
+    name="camera_left_ir_optical_frame">
     <inertial>
       <origin
@@ -298,5 +298,5 @@
   </link>
   <joint
-    name="camera_infra1_optical_frame"
+    name="camera_left_ir_optical_frame"
     type="fixed">
     <origin
@@ -304,12 +304,12 @@
       rpy="-1.5708 0 -1.5708" />
     <parent
-      link="camera_infra1_frame" />
-    <child
-      link="camera_infra1_optical_frame" />
-    <axis
-      xyz="0 0 0" />
-  </joint>
-  <link
-    name="camera_infra2_frame">
+      link="camera_left_ir_frame" />
+    <child
+      link="camera_left_ir_optical_frame" />
+    <axis
+      xyz="0 0 0" />
+  </joint>
+  <link
+    name="camera_right_ir_frame">
     <inertial>
       <origin
@@ -351,18 +351,18 @@
   </link>
   <joint
-    name="camera_infra2_frame"
-    type="fixed">
-    <origin
-      xyz="0.011715 -0.0475 0.014311"
+    name="camera_right_ir_frame"
+    type="fixed">
+    <origin
+      xyz="0 -0.095 0"
       rpy="0 0 0" />
     <parent
-      link="camera_color_screw_frame" />
-    <child
-      link="camera_infra2_frame" />
-    <axis
-      xyz="0 0 0" />
-  </joint>
-  <link
-    name="camera_infra2_optical_frame">
+      link="camera_depth_frame" />
+    <child
+      link="camera_right_ir_frame" />
+    <axis
+      xyz="0 0 0" />
+  </joint>
+  <link
+    name="camera_right_ir_optical_frame">
     <inertial>
       <origin
@@ -404,5 +404,5 @@
   </link>
   <joint
-    name="camera_infra2_optical_frame"
+    name="camera_right_ir_optical_frame"
     type="fixed">
     <origin
@@ -410,7 +410,7 @@
       rpy="-1.5708 0 -1.5708" />
     <parent
-      link="camera_infra2_frame" />
-    <child
-      link="camera_infra2_optical_frame" />
+      link="camera_right_ir_frame" />
+    <child
+      link="camera_right_ir_optical_frame" />
     <axis
       xyz="0 0 0" />
@@ -460,8 +460,8 @@
     type="fixed">
     <origin
-      xyz="0.011715 0.02375 0.014311"
+      xyz="0 -0.02375 0"
       rpy="0.0010157 0 0" />
     <parent
-      link="camera_color_screw_frame" />
+      link="camera_depth_frame" />
     <child
       link="camera_color_frame" />

File: urdf/gemini335Le.urdf.xacro (robot description, xacro)
@@ -5,5 +5,5 @@
      For more information, please see http://wiki.ros.org/sw_urdf_exporter -->
 <robot xmlns:xacro="http://ros.org/wiki/xacro" name="gemini335Le">
-    <xacro:property name="mesh_path" value="package://orbbec_camera/meshes/gemini335Le/" />
+    <xacro:property name="mesh_path" value="package://orbbec_description/meshes/gemini335Le/" />
    <link
     name="camera_link">
@@ -24,5 +24,5 @@
     <visual>
       <origin
-        xyz="0 0 0"
+        xyz="-0.034005 -0.0475 -0.014048"
         rpy="0 0 0" />
       <geometry>
@@ -86,19 +86,6 @@
     </collision>
   </link>
-  <joint
-    name="base_Joint"
-    type="fixed">
-    <origin
-      xyz="0 0 0"
-      rpy="0 0 0" />
-    <parent
-      link="camera_botton_screw_frame" />
-    <child
-      link="camera_link" />
-    <axis
-      xyz="0 0 0" />
-  </joint>
-  <link
-    name="canera_right_IR_ROS_frame">
+    <link
+    name="camera_depth_frame">
     <inertial>
       <origin
@@ -115,43 +102,33 @@
         izz="4.8408E-09" />
     </inertial>
-    <visual>
-      <origin
-        xyz="0 0 0"
-        rpy="0 0 0" />
-      <geometry>
-        <mesh
-          filename="${mesh_path}canera_right_IR_ROS_frame.STL" />
-      </geometry>
-      <material
-        name="">
-        <color
-          rgba="0.3 0.3 0.3 1" />
-      </material>
-    </visual>
-    <collision>
-      <origin
-        xyz="0 0 0"
-        rpy="0 0 0" />
-      <geometry>
-        <mesh
-          filename="${mesh_path}canera_right_IR_ROS_frame.STL" />
-      </geometry>
-    </collision>
-  </link>
-  <joint
-    name="canera_right_IR_ROS_Joint"
-    type="fixed">
-    <origin
-      xyz="0.034005 -0.0475 0.014048"
+  </link>
+  <joint
+    name="camera_depth_frame_Joint"
+    type="fixed">
+    <origin
+      xyz="0 0 0"
       rpy="0 0 0" />
     <parent
       link="camera_link" />
     <child
-      link="canera_right_IR_ROS_frame" />
+      link="camera_depth_frame" />
+    <axis
+      xyz="0 0 0" />
+  </joint>
+  <joint
+    name="base_Joint"
+    type="fixed">
+    <origin
+      xyz="-0.034005 -0.0475 -0.014048"
+      rpy="0 0 0" />
+    <parent
+      link="camera_link" />
+    <child
+      link="camera_botton_screw_frame" />
     <axis
       xyz="0 0 0" />
   </joint>
   <link
-    name="canera_left_IR_ROS_frame">
+    name="camera_right_ir_frame">
     <inertial>
       <origin
@@ -174,4 +151,57 @@
       <geometry>
         <mesh
+          filename="${mesh_path}canera_right_IR_ROS_frame.STL" />
+      </geometry>
+      <material
+        name="">
+        <color
+          rgba="0.3 0.3 0.3 1" />
+      </material>
+    </visual>
+    <collision>
+      <origin
+        xyz="0 0 0"
+        rpy="0 0 0" />
+      <geometry>
+        <mesh
+          filename="${mesh_path}canera_right_IR_ROS_frame.STL" />
+      </geometry>
+    </collision>
+  </link>
+  <joint
+    name="camera_right_ir_Joint"
+    type="fixed">
+    <origin
+      xyz="0 -0.095 0"
+      rpy="0 0 0" />
+    <parent
+      link="camera_depth_frame" />
+    <child
+      link="camera_right_ir_frame" />
+    <axis
+      xyz="0 0 0" />
+  </joint>
+  <link
+    name="camera_left_ir_frame">
+    <inertial>
+      <origin
+        xyz="-0.0015782 9.8699E-08 -1.6899E-07"
+        rpy="0 0 0" />
+      <mass
+        value="0.00045313" />
+      <inertia
+        ixx="4.3406E-09"
+        ixy="-5.1012E-13"
+        ixz="-6.3511E-13"
+        iyy="4.8388E-09"
+        iyz="1.081E-12"
+        izz="4.8408E-09" />
+    </inertial>
+    <visual>
+      <origin
+        xyz="0 0 0"
+        rpy="0 0 0" />
+      <geometry>
+        <mesh
           filename="${mesh_path}canera_left_IR_ROS_frame.STL" />
       </geometry>
@@ -193,18 +223,18 @@
   </link>
   <joint
-    name="canera_left_IR_ROS_Joint"
-    type="fixed">
-    <origin
-      xyz="0.034005 0.0475 0.014048"
-      rpy="0 0 0" />
-    <parent
-      link="camera_link" />
-    <child
-      link="canera_left_IR_ROS_frame" />
+    name="camera_left_ir_Joint"
+    type="fixed">
+    <origin
+      xyz="0 0 0"
+      rpy="0 0 0" />
+    <parent
+      link="camera_depth_frame" />
+    <child
+      link="camera_left_ir_frame" />
     <axis
       xyz="0 0 0" />
   </joint>
   <link
-    name="canera_RGB_ROS_frame">
+    name="camera_color_frame">
     <inertial>
       <origin
@@ -246,18 +276,18 @@
   </link>
   <joint
-    name="canera_RGB_ROS_Joint"
-    type="fixed">
-    <origin
-      xyz="0.034014 0.02375 0.014048"
-      rpy="0 0 0" />
-    <parent
-      link="camera_link" />
-    <child
-      link="canera_RGB_ROS_frame" />
+    name="camera_color_Joint"
+    type="fixed">
+    <origin
+      xyz="9e-06 -0.02375 0"
+      rpy="0 0 0" />
+    <parent
+      link="camera_depth_frame" />
+    <child
+      link="camera_color_frame" />
     <axis
       xyz="0 0 0" />
   </joint>
   <link
-    name="canera_IMU_ROS_frame">
+    name="camera_imu_frame">
     <inertial>
       <origin
@@ -299,13 +329,13 @@
   </link>
   <joint
-    name="canera_IMU_ROS_Joint"
-    type="fixed">
-    <origin
-      xyz="0.019757 0.03619 0.013358"
-      rpy="0 0 0" />
-    <parent
-      link="camera_link" />
-    <child
-      link="canera_IMU_ROS_frame" />
+    name="camera_imu_Joint"
+    type="fixed">
+    <origin
+      xyz="-0.014248 -0.01131 -0.00069"
+      rpy="0 0 0" />
+    <parent
+      link="camera_depth_frame" />
+    <child
+      link="camera_imu_frame" />
     <axis
       xyz="0 0 0" />
