Commit message: Refactor URDF files for camera frames and joints

File: urdf/gemini335Lg.urdf.xacro (robot description, xacro)
@@ -5,5 +5,5 @@
      For more information, please see http://wiki.ros.org/sw_urdf_exporter -->
 <robot xmlns:xacro="http://ros.org/wiki/xacro" name="gemini335_336Lg">
-    <xacro:property name="mesh_path" value="package://orbbec_camera/meshes/gemini335Lg/" />
+    <xacro:property name="mesh_path" value="package://orbbec_description/meshes/gemini335Lg/" />
     <link
     name="camera_link">
@@ -24,5 +24,5 @@
     <visual>
       <origin
-        xyz="0 0 0"
+        xyz="-0.0117149999999995 -0.0475 -0.0143111800025738"
         rpy="0 0 0" />
       <geometry>
@@ -90,5 +90,5 @@
     type="fixed">
     <origin
-      xyz="0 0 0"
+      xyz="-0.0117149999999995 -0.0475 -0.0143111800025738"
       rpy="0 0 0" />
     <parent
@@ -100,5 +100,5 @@
   </joint>
   <link
-    name="camera_infra1_frame">
+    name="camera_left_ir_frame">
     <inertial>
       <origin
@@ -140,18 +140,18 @@
   </link>
   <joint
-    name="camera_infra1_frame"
-    type="fixed">
-    <origin
-      xyz="0.0117149999999995 0.0475 0.0143111800025738"
+    name="camera_left_ir_frame"
+    type="fixed">
+    <origin
+      xyz="0 0 0"
       rpy="0 0 0" />
     <parent
-      link="camera_bottom_screw_frame" />
-    <child
-      link="camera_infra1_frame" />
-    <axis
-      xyz="0 0 0" />
-  </joint>
-  <link
-    name="camera_infra1_optical_frame">
+      link="camera_depth_frame" />
+    <child
+      link="camera_left_ir_frame" />
+    <axis
+      xyz="0 0 0" />
+  </joint>
+  <link
+    name="camera_left_ir_optical_frame">
     <inertial>
       <origin
@@ -193,5 +193,5 @@
   </link>
   <joint
-    name="camera_infra1_optical_frame"
+    name="camera_left_ir_optical_frame"
     type="fixed">
     <origin
@@ -199,7 +199,7 @@
       rpy="-1.5707963267949 0 -1.5707963267949" />
     <parent
-      link="camera_infra1_frame" />
-    <child
-      link="camera_infra1_optical_frame" />
+      link="camera_left_ir_frame" />
+    <child
+      link="camera_left_ir_optical_frame" />
     <axis
       xyz="0 0 0" />
@@ -249,8 +249,8 @@
     type="fixed">
     <origin
-      xyz="0.0117149999999995 0.02375 0.0143111800025738"
+      xyz="0 -0.023749999701976776 0"
       rpy="0 0 0" />
     <parent
-      link="camera_bottom_screw_frame" />
+      link="camera_depth_frame" />
     <child
       link="camera_color_frame" />
@@ -312,5 +312,5 @@
   </joint>
   <link
-    name="camera_infra2_frame">
+    name="camera_right_ir_frame">
     <inertial>
       <origin
@@ -352,18 +352,18 @@
   </link>
   <joint
-    name="camera_infra2_frame"
-    type="fixed">
-    <origin
-      xyz="0.0117149999999995 -0.0475 0.0143111800025738"
+    name="camera_right_ir_frame"
+    type="fixed">
+    <origin
+      xyz="0 -0.095 0"
       rpy="0 0 0" />
     <parent
-      link="camera_bottom_screw_frame" />
-    <child
-      link="camera_infra2_frame" />
-    <axis
-      xyz="0 0 0" />
-  </joint>
-  <link
-    name="camera_infra2_optical_frame">
+      link="camera_depth_frame" />
+    <child
+      link="camera_right_ir_frame" />
+    <axis
+      xyz="0 0 0" />
+  </joint>
+  <link
+    name="camera_right_ir_optical_frame">
     <inertial>
       <origin
@@ -405,5 +405,5 @@
   </link>
   <joint
-    name="camera_infra2_optical_frame"
+    name="camera_right_ir_optical_frame"
     type="fixed">
     <origin
@@ -411,12 +411,12 @@
       rpy="-1.57079632679486 0 -1.5707963267949" />
     <parent
-      link="camera_infra2_frame" />
-    <child
-      link="camera_infra2_optical_frame" />
-    <axis
-      xyz="0 0 0" />
-  </joint>
-  <link
-    name="camera_IMU_frame">
+      link="camera_right_ir_frame" />
+    <child
+      link="camera_right_ir_optical_frame" />
+    <axis
+      xyz="0 0 0" />
+  </joint>
+  <link
+    name="camera_imu_frame">
     <inertial>
       <origin
@@ -458,13 +458,13 @@
   </link>
   <joint
-    name="camera_IMU_frame"
-    type="fixed">
-    <origin
-      xyz="-0.00253500000000046 0.036187989999999 0.0136240800025733"
+    name="camera_imu_frame"
+    type="fixed">
+    <origin
+      xyz="-0.01425 -0.011312 -0.0006871"
       rpy="0 0 0" />
     <parent
-      link="camera_bottom_screw_frame" />
-    <child
-      link="camera_IMU_frame" />
+      link="camera_depth_frame" />
+    <child
+      link="camera_imu_frame" />
     <axis
       xyz="0 0 0" />
@@ -514,8 +514,8 @@
     type="fixed">
     <origin
-      xyz="0.0117149999999995 0.0475 0.0143111800025738"
+      xyz="0 0 0"
       rpy="0 0 0" />
     <parent
-      link="camera_bottom_screw_frame" />
+      link="camera_link" />
     <child
       link="camera_depth_frame" />

File: urdf/gemini_335_336.urdf.xacro (robot description, xacro)
@@ -4,6 +4,6 @@
      Commit Version: 1.6.0-4-g7f85cfe  Build Version: 1.6.7995.38578
      For more information, please see http://wiki.ros.org/sw_urdf_exporter -->
-<robot xmlns:xacro="http://ros.org/wiki/xacro" name="gemini335_336">
-    <xacro:property name="mesh_path" value="package://orbbec_camera/meshes/gemini335_336/" />
+<robot xmlns:xacro="http://ros.org/wiki/xacro" name="gemini_335_336">
+    <xacro:property name="mesh_path" value="package://orbbec_description/meshes/gemini335_336/" />
     <link name="camera_link">
         <inertial>
@@ -15,5 +15,5 @@
         </inertial>
         <visual>
-            <origin xyz="0 0 0" rpy="0 0 0" />
+            <origin xyz="-0.01587 -0.025 -0.0125" rpy="0 0 0" />
             <geometry>
                 <mesh filename="${mesh_path}camera_link.STL" />
@@ -55,5 +55,5 @@
     </link>
     <joint name="camera_bottom_screw_frame_joint" type="fixed">
-        <origin xyz="0 0 0" rpy="0 0 0" />
+        <origin xyz="-0.01587 -0.025 -0.0125" rpy="0 0 0" />
         <parent link="camera_link" />
         <child link="camera_bottom_screw_frame" />
@@ -86,6 +86,6 @@
     </link>
     <joint name="camera_left_ir_joint" type="fixed">
-        <origin xyz="0.01587 -0.025 0.0125" rpy="0 0 0" />
-        <parent link="camera_bottom_screw_frame" />
+        <origin xyz="0 0 0" rpy="0 0 0" />
+        <parent link="camera_depth_frame" />
         <child link="camera_left_ir_frame" />
         <axis xyz="0 0 0" />
@@ -116,6 +116,6 @@
     </link>
     <joint name="camera_left_ir_optical_joint" type="fixed">
-        <origin xyz="0.01587 -0.025 0.0125" rpy="-1.5707963267949 0 -1.5707963267949" />
-        <parent link="camera_bottom_screw_frame" />
+        <origin xyz="0 0 0" rpy="-1.5707963267949 0 -1.5707963267949" />
+        <parent link="camera_left_ir_frame" />
         <child link="camera_left_ir_optical_frame" />
         <axis xyz="0 0 0" />
@@ -147,6 +147,6 @@
     </link>
     <joint name="camera_right_ir_joint" type="fixed">
-        <origin xyz="0.01587 0.025 0.0125" rpy="0 0 0" />
-        <parent link="camera_bottom_screw_frame" />
+        <origin xyz="0 -0.05 0" rpy="0 0 0" />
+        <parent link="camera_depth_frame" />
         <child link="camera_right_ir_frame" />
         <axis xyz="0 0 0" />
@@ -177,6 +177,6 @@
     </link>
     <joint name="camera_right_ir_optical_joint" type="fixed">
-        <origin xyz="0.01587 0.025 0.0125" rpy="-1.5707963267949 0 -1.5707963267949" />
-        <parent link="camera_bottom_screw_frame" />
+        <origin xyz="0 0 0" rpy="-1.5707963267949 0 -1.5707963267949" />
+        <parent link="camera_right_ir_frame" />
         <child link="camera_right_ir_optical_frame" />
         <axis xyz="0 0 0" />
@@ -208,6 +208,6 @@
     </link>
     <joint name="camera_color_joint" type="fixed">
-        <origin xyz="0.017533 0.010995 0.012505" rpy="0 0 0" />
-        <parent link="camera_bottom_screw_frame" />
+        <origin xyz="0.001663 -0.014005 0.000005" rpy="0 0 0" />
+        <parent link="camera_depth_frame" />
         <child link="camera_color_frame" />
         <axis xyz="0 0 0" />
@@ -239,6 +239,6 @@
     </link>
     <joint name="camera_color_optical_joint" type="fixed">
-        <origin xyz="0.017533 0.010995 0.012505" rpy="-1.5707963267949 0 -1.5707963267949" />
-        <parent link="camera_bottom_screw_frame" />
+        <origin xyz="0 0 0" rpy="-1.5707963267949 0 -1.5707963267949" />
+        <parent link="camera_color_frame" />
         <child link="camera_color_optical_frame" />
         <axis xyz="0 0 0" />
@@ -270,6 +270,6 @@
     </link>
     <joint name="camera_depth_joint" type="fixed">
-        <origin xyz="0.01587 -0.025 0.0125" rpy="0 0 0" />
-        <parent link="camera_bottom_screw_frame" />
+        <origin xyz="0 0 0" rpy="0 0 0" />
+        <parent link="camera_link" />
         <child link="camera_depth_frame" />
         <axis xyz="0 0 0" />
@@ -299,6 +299,6 @@
     </link>
     <joint name="camera_depth_optical_joint" type="fixed">
-        <origin xyz="0.01587 -0.025 0.0125" rpy="-1.5707963267949 0 -1.5707963267949" />
-        <parent link="camera_bottom_screw_frame" />
+        <origin xyz="0 0 0" rpy="-1.5707963267949 0 -1.5707963267949" />
+        <parent link="camera_depth_frame" />
         <child link="camera_depth_optical_frame" />
         <axis xyz="0 0 0" />

File: urdf/test_astra2.urdf.xacro (robot description, xacro)
@@ -4,5 +4,5 @@
      For more information, please see http://wiki.ros.org/sw_urdf_exporter -->
 <robot name="astra2" xmlns:xacro="http://ros.org/wiki/xacro">
-    <xacro:include filename="astra2.urdf.xarco"/>
+    <xacro:include filename="astra2.urdf.xacro"/>
     <!-- Define a virtual root link -->
   <link name="base_link"/>
@@ -11,5 +11,5 @@
     <parent link="base_link"/>
     <child link="camera_link"/>
-    <origin xyz="0 0 0" rpy="0 0 0"/>
+    <origin xyz="0.012323996052145958 0.03750000149011612 0.028150320053100586" rpy="0 0 0"/>
   </joint>
 </robot>

File: urdf/test_gemini2.urdf.xacro (robot description, xacro)
@@ -3,6 +3,6 @@
      Commit Version: 1.6.0-4-g7f85cfe  Build Version: 1.6.7995.38578
      For more information, please see http://wiki.ros.org/sw_urdf_exporter -->
-<robot name="gemini335Le" xmlns:xacro="http://ros.org/wiki/xacro">
-    <xacro:include filename="gemini335Le.urdf.xacro"/>
+<robot name="gemini2" xmlns:xacro="http://ros.org/wiki/xacro">
+    <xacro:include filename="gemini2.urdf.xacro"/>
     <!-- Define a virtual root link -->
   <link name="base_link"/>
@@ -10,6 +10,6 @@
   <joint name="base_link_to_camera_link" type="fixed">
     <parent link="base_link"/>
-    <child link="camera_botton_screw_frame"/>
-    <origin xyz="0 0 0" rpy="0 0 0"/>
+    <child link="camera_link"/>
+    <origin xyz="0.01491 0.025 0.0125" rpy="0 0 0"/>
   </joint>
 </robot>

File: urdf/test_gemini2L.urdf.xacro (robot description, xacro)
@@ -3,6 +3,6 @@
      Commit Version: 1.6.0-4-g7f85cfe  Build Version: 1.6.7995.38578
      For more information, please see http://wiki.ros.org/sw_urdf_exporter -->
-<robot name="gemini335Lg" xmlns:xacro="http://ros.org/wiki/xacro">
-    <xacro:include filename="gemini335Lg.urdf.xacro"/>
+<robot name="gemini2L" xmlns:xacro="http://ros.org/wiki/xacro">
+    <xacro:include filename="gemini2L.urdf.xacro"/>
     <!-- Define a virtual root link -->
   <link name="base_link"/>
@@ -11,5 +11,5 @@
     <parent link="base_link"/>
     <child link="camera_link"/>
-    <origin xyz="0 0 0" rpy="0 0 0"/>
+    <origin xyz="0.01033 0.05 0.0145" rpy="0 0 0"/>
   </joint>
 </robot>

File: urdf/test_gemini335L.urdf.xacro (robot description, xacro)
@@ -3,6 +3,6 @@
      Commit Version: 1.6.0-4-g7f85cfe  Build Version: 1.6.7995.38578
      For more information, please see http://wiki.ros.org/sw_urdf_exporter -->
-<robot name="gemini335" xmlns:xacro="http://ros.org/wiki/xacro">
-    <xacro:include filename="gemini335_336.urdf.xacro"/>
+<robot name="gemini335L" xmlns:xacro="http://ros.org/wiki/xacro">
+    <xacro:include filename="gemini335L_336L.urdf.xacro"/>
     <!-- Define a virtual root link -->
   <link name="base_link"/>
@@ -11,5 +11,5 @@
     <parent link="base_link"/>
     <child link="camera_link"/>
-    <origin xyz="0 0 0" rpy="0 0 0"/>
+    <origin xyz="0.011715 0.0475 0.014311" rpy="0 0 0"/>
   </joint>
 </robot>

File: urdf/test_gemini335Le.urdf.xacro (robot description, xacro)
@@ -3,6 +3,6 @@
      Commit Version: 1.6.0-4-g7f85cfe  Build Version: 1.6.7995.38578
      For more information, please see http://wiki.ros.org/sw_urdf_exporter -->
-<robot name="gemini336L" xmlns:xacro="http://ros.org/wiki/xacro">
-    <xacro:include filename="gemini335L_336L.urdf.xarco"/>
+<robot name="gemini335Le" xmlns:xacro="http://ros.org/wiki/xacro">
+    <xacro:include filename="gemini335Le.urdf.xacro"/>
     <!-- Define a virtual root link -->
   <link name="base_link"/>
@@ -11,5 +11,5 @@
     <parent link="base_link"/>
     <child link="camera_link"/>
-    <origin xyz="0 0 0" rpy="0 0 0"/>
+    <origin xyz="0.034005 0.0475 0.014048" rpy="0 0 0"/>
   </joint>
 </robot>

File: urdf/test_gemini335Lg.urdf.xacro (robot description, xacro)
@@ -3,6 +3,6 @@
      Commit Version: 1.6.0-4-g7f85cfe  Build Version: 1.6.7995.38578
      For more information, please see http://wiki.ros.org/sw_urdf_exporter -->
-<robot name="gemini2" xmlns:xacro="http://ros.org/wiki/xacro">
-    <xacro:include filename="gemini2.urdf.xarco"/>
+<robot name="gemini335Lg" xmlns:xacro="http://ros.org/wiki/xacro">
+    <xacro:include filename="gemini335Lg.urdf.xacro"/>
     <!-- Define a virtual root link -->
   <link name="base_link"/>
@@ -11,5 +11,5 @@
     <parent link="base_link"/>
     <child link="camera_link"/>
-    <origin xyz="0 0 0" rpy="0 0 0"/>
+    <origin xyz="0.0117149999999995 0.0475 0.0143111800025738" rpy="0 0 0"/>
   </joint>
 </robot>

File: urdf/test_gemini336L.urdf.xacro (robot description, xacro)
@@ -3,6 +3,6 @@
      Commit Version: 1.6.0-4-g7f85cfe  Build Version: 1.6.7995.38578
      For more information, please see http://wiki.ros.org/sw_urdf_exporter -->
-<robot name="gemini2L" xmlns:xacro="http://ros.org/wiki/xacro">
-    <xacro:include filename="gemini2L.urdf.xarco"/>
+<robot name="gemini336L" xmlns:xacro="http://ros.org/wiki/xacro">
+    <xacro:include filename="gemini335L_336L.urdf.xacro"/>
     <!-- Define a virtual root link -->
   <link name="base_link"/>
@@ -11,5 +11,5 @@
     <parent link="base_link"/>
     <child link="camera_link"/>
-    <origin xyz="0 0 0" rpy="0 0 0"/>
+    <origin xyz="0.011715 0.0475 0.014311" rpy="0 0 0"/>
   </joint>
 </robot>

Commit message: fix: update mesh paths in URDF files to point to the correct package location

File: urdf/astra2.urdf.xacro (robot description, xacro)
@@ -4,5 +4,5 @@
      For more information, please see http://wiki.ros.org/sw_urdf_exporter -->
 <robot xmlns:xacro="http://ros.org/wiki/xacro" name="astra2">
-    <xacro:property name="mesh_path" value="package://orbbec_description/meshes/astra2/" />
+    <xacro:property name="mesh_path" value="package://orbbec_camera/meshes/astra2/" />
   <link
     name="camera_link">

File: urdf/femto_bolt.urdf.xacro (robot description, xacro)
@@ -11,5 +11,5 @@
   <xacro:property name="cam_height" value="0.06495"/>
   <xacro:property name="cam_depth" value="0.04026"/>
-  <xacro:property name="mesh_path" value="package://orbbec_description/meshes/femto_bolt/" />
+  <xacro:property name="mesh_path" value="package://orbbec_camera/meshes/femto_bolt/" />
   <!-- The following values are approximate but the camera node
      publishes TF values with actual calibrated camera extrinsic values -->

File: urdf/gemini2.urdf.xacro (robot description, xacro)
@@ -4,5 +4,5 @@
      For more information, please see http://wiki.ros.org/sw_urdf_exporter -->
 <robot xmlns:xacro="http://ros.org/wiki/xacro" name="gemini2">
-    <xacro:property name="mesh_path" value="package://orbbec_description/meshes/gemini2/" />
+    <xacro:property name="mesh_path" value="package://orbbec_camera/meshes/gemini2/" />
   <link
     name="camera_link">

File: urdf/gemini2L.urdf.xacro (robot description, xacro)
@@ -4,5 +4,5 @@
      For more information, please see http://wiki.ros.org/sw_urdf_exporter -->
 <robot xmlns:xacro="http://ros.org/wiki/xacro" name="gemini2l">
-    <xacro:property name="mesh_path" value="package://orbbec_description/meshes/gemini2l/" />
+    <xacro:property name="mesh_path" value="package://orbbec_camera/meshes/gemini2l/" />
   <link
     name="camera_link">

File: urdf/gemini335L_336L.urdf.xacro (robot description, xacro)
@@ -4,5 +4,5 @@
      For more information, please see http://wiki.ros.org/sw_urdf_exporter -->
 <robot xmlns:xacro="http://ros.org/wiki/xacro" name="gemini_335L_336L">
-    <xacro:property name="mesh_path" value="package://orbbec_description/meshes/gemini335L_336L/" />
+    <xacro:property name="mesh_path" value="package://orbbec_camera/meshes/gemini335L_336L/" />
   <link
     name="camera_link">

File: urdf/gemini335Le.urdf.xacro (robot description, xacro)
@@ -5,5 +5,5 @@
      For more information, please see http://wiki.ros.org/sw_urdf_exporter -->
 <robot xmlns:xacro="http://ros.org/wiki/xacro" name="gemini335Le">
-    <xacro:property name="mesh_path" value="package://orbbec_description/meshes/gemini335Le/" />
+    <xacro:property name="mesh_path" value="package://orbbec_camera/meshes/gemini335Le/" />
    <link
     name="camera_link">

File: urdf/gemini335Lg.urdf.xacro (robot description, xacro)
@@ -5,5 +5,5 @@
      For more information, please see http://wiki.ros.org/sw_urdf_exporter -->
 <robot xmlns:xacro="http://ros.org/wiki/xacro" name="gemini335_336Lg">
-    <xacro:property name="mesh_path" value="package://orbbec_description/meshes/gemini335Lg/" />
+    <xacro:property name="mesh_path" value="package://orbbec_camera/meshes/gemini335Lg/" />
     <link
     name="camera_link">

File: urdf/gemini_335_336.urdf.xacro (robot description, xacro)
@@ -5,5 +5,5 @@
      For more information, please see http://wiki.ros.org/sw_urdf_exporter -->
 <robot xmlns:xacro="http://ros.org/wiki/xacro" name="gemini_335_336">
-    <xacro:property name="mesh_path" value="package://orbbec_description/meshes/gemini335_336/" />
+    <xacro:property name="mesh_path" value="package://orbbec_camera/meshes/gemini335_336/" />
     <link name="camera_link">
         <inertial>
