Commit message: Refactor URDF files for camera frames and joints

File: urdf/astra2.urdf.xacro (robot description, xacro)
@@ -23,5 +23,5 @@
     <visual>
       <origin
-        xyz="0 0 0"
+        xyz="-0.012323995999904 -0.0374999999985815 -0.0281503197112"
         rpy="0 0 0" />
       <geometry>
@@ -89,5 +89,5 @@
     type="fixed">
     <origin
-      xyz="0 0 0"
+      xyz="-0.012323995999904 -0.0374999999985815 -0.0281503197112"
       rpy="0 0 0" />
     <parent
@@ -99,5 +99,5 @@
   </joint>
   <link
-    name="camera_infra1_frame">
+    name="camera_ir_frame">
     <inertial>
       <origin
@@ -139,18 +139,18 @@
   </link>
   <joint
-    name="camera_infra1_frame"
-    type="fixed">
-    <origin
-      xyz="0.012323995999904 0.0374999999985815 0.0281503197112"
+    name="camera_ir_frame"
+    type="fixed">
+    <origin
+      xyz="0 0 0"
       rpy="0 0 0" />
     <parent
-      link="camera_bottom_screw_frame" />
-    <child
-      link="camera_infra1_frame" />
-    <axis
-      xyz="0 0 0" />
-  </joint>
-  <link
-    name="camera_infra1_optical_frame">
+      link="camera_depth_frame" />
+    <child
+      link="camera_ir_frame" />
+    <axis
+      xyz="0 0 0" />
+  </joint>
+  <link
+    name="camera_ir_optical_frame">
     <inertial>
       <origin
@@ -192,5 +192,5 @@
   </link>
   <joint
-    name="camera_infra1_optical_frame"
+    name="camera_ir_optical_frame"
     type="fixed">
     <origin
@@ -198,12 +198,12 @@
       rpy="-1.5707963267949 0 -1.5707963267949" />
     <parent
-      link="camera_infra1_frame" />
-    <child
-      link="camera_infra1_optical_frame" />
-    <axis
-      xyz="0 0 0" />
-  </joint>
-  <link
-    name="camera_colorl_frame">
+      link="camera_ir_frame" />
+    <child
+      link="camera_ir_optical_frame" />
+    <axis
+      xyz="0 0 0" />
+  </joint>
+  <link
+    name="camera_color_frame">
     <inertial>
       <origin
@@ -248,10 +248,10 @@
     type="fixed">
     <origin
-      xyz="0.014865995999904 0.0189999999985815 0.0281503197112"
+      xyz="0.0025420000310987234 -0.01850000023841858 0"
       rpy="0 0 0" />
     <parent
-      link="camera_bottom_screw_frame" />
-    <child
-      link="camera_colorl_frame" />
+      link="camera_depth_frame" />
+    <child
+      link="camera_color_frame" />
     <axis
       xyz="0 0 0" />
@@ -304,5 +304,5 @@
       rpy="-1.5707963267949 0 -1.5707963267949" />
     <parent
-      link="camera_colorl_frame" />
+      link="camera_color_frame" />
     <child
       link="camera_color_optical_frame" />
@@ -354,8 +354,8 @@
     type="fixed">
     <origin
-      xyz="0.012323995999904 0.0374999999985815 0.0281503197112"
+      xyz="0 0 0"
       rpy="0 0 0" />
     <parent
-      link="camera_bottom_screw_frame" />
+      link="camera_link" />
     <child
       link="camera_depth_frame" />

File: urdf/gemini2.urdf.xacro (robot description, xacro)
@@ -23,5 +23,5 @@
     <visual>
       <origin
-        xyz="0 0 0"
+        xyz="-0.01491 -0.025 -0.0125"
         rpy="0 0 0" />
       <geometry>
@@ -89,5 +89,5 @@
     type="fixed">
     <origin
-      xyz="0 0 0"
+      xyz="-0.01491 -0.025 -0.0125"
       rpy="0 0 0" />
     <parent
@@ -99,5 +99,5 @@
   </joint>
   <link
-    name="camera_infra1_frame">
+    name="camera_right_ir_frame">
     <inertial>
       <origin
@@ -139,18 +139,18 @@
   </link>
   <joint
-    name="camera_infra1_frame"
-    type="fixed">
-    <origin
-      xyz="0.01491 -0.025 0.0125"
+    name="camera_right_ir_frame"
+    type="fixed">
+    <origin
+      xyz="0 -0.05000000074505806 0"
       rpy="0 0 0" />
     <parent
-      link="camera_botter_screw_frame" />
-    <child
-      link="camera_infra1_frame" />
-    <axis
-      xyz="0 0 0" />
-  </joint>
-  <link
-    name="camera_infra1_optical_frame">
+      link="camera_depth_frame" />
+    <child
+      link="camera_right_ir_frame" />
+    <axis
+      xyz="0 0 0" />
+  </joint>
+  <link
+    name="camera_right_ir_optical_frame">
     <inertial>
       <origin
@@ -192,5 +192,5 @@
   </link>
   <joint
-    name="camera_infra1_optical_frame"
+    name="camera_right_ir_optical_frame"
     type="fixed">
     <origin
@@ -198,7 +198,7 @@
       rpy="-1.5707963267949 0 -1.5707963267949" />
     <parent
-      link="camera_infra1_frame" />
-    <child
-      link="camera_infra1_optical_frame" />
+      link="camera_right_ir_frame" />
+    <child
+      link="camera_right_ir_optical_frame" />
     <axis
       xyz="0 0 0" />
@@ -248,8 +248,8 @@
     type="fixed">
     <origin
-      xyz="0.01682 0.010995 0.012505"
-      rpy="-1.5707963267949 0 -1.5707963267949" />
-    <parent
-      link="camera_botter_screw_frame" />
+      xyz="0.0019099999917671084 -0.01400499977171421 4.999999873689376e-06"
+      rpy="0 0 0" />
+    <parent
+      link="camera_depth_frame" />
     <child
       link="camera_color_frame" />
@@ -302,5 +302,5 @@
     <origin
       xyz="0 0 0"
-      rpy="0 0 0" />
+      rpy="-1.5707963267949 0 -1.5707963267949" />
     <parent
       link="camera_color_frame" />
@@ -311,5 +311,5 @@
   </joint>
   <link
-    name="camera_infra2_frame">
+    name="camera_left_ir_frame">
     <inertial>
       <origin
@@ -351,18 +351,18 @@
   </link>
   <joint
-    name="camera_infra2_frame"
-    type="fixed">
-    <origin
-      xyz="0.01491 0.025 0.0125"
+    name="camera_left_ir_frame"
+    type="fixed">
+    <origin
+      xyz="0 0 0"
       rpy="0 0 0" />
     <parent
-      link="camera_botter_screw_frame" />
-    <child
-      link="camera_infra2_frame" />
-    <axis
-      xyz="0 0 0" />
-  </joint>
-  <link
-    name="camera_infra2_optical_frame">
+      link="camera_link" />
+    <child
+      link="camera_left_ir_frame" />
+    <axis
+      xyz="0 0 0" />
+  </joint>
+  <link
+    name="camera_left_ir_optical_frame">
     <inertial>
       <origin
@@ -404,5 +404,5 @@
   </link>
   <joint
-    name="camera_infra2_optical_frame"
+    name="camera_left_ir_optical_frame"
     type="fixed">
     <origin
@@ -410,7 +410,7 @@
       rpy="-1.5707963267949 0 -1.5707963267949" />
     <parent
-      link="camera_infra2_frame" />
-    <child
-      link="camera_infra2_optical_frame" />
+      link="camera_left_ir_frame" />
+    <child
+      link="camera_left_ir_optical_frame" />
     <axis
       xyz="0 0 0" />
@@ -460,8 +460,8 @@
     type="fixed">
     <origin
-      xyz="0.01491 0.025 0.0125"
+      xyz="0 0 0"
       rpy="0 0 0" />
     <parent
-      link="camera_botter_screw_frame" />
+      link="camera_link" />
     <child
       link="camera_depth_frame" />

File: urdf/gemini2L.urdf.xacro (robot description, xacro)
@@ -23,5 +23,5 @@
     <visual>
       <origin
-        xyz="0 0 0"
+        xyz="-0.01033 -0.05 -0.0145"
         rpy="0 0 0" />
       <geometry>
@@ -89,5 +89,5 @@
     type="fixed">
     <origin
-      xyz="0 0 0"
+      xyz="-0.01033 -0.05 -0.0145"
       rpy="0 0 0" />
     <parent
@@ -99,5 +99,5 @@
   </joint>
   <link
-    name="camera_IR2_frame">
+    name="camera_right_ir_frame">
     <inertial>
       <origin
@@ -139,18 +139,18 @@
   </link>
   <joint
-    name="camera_IR2_frame"
-    type="fixed">
-    <origin
-      xyz="0.01033 -0.05 0.0145"
+    name="camera_right_ir_frame"
+    type="fixed">
+    <origin
+      xyz="0 -0.1 0"
       rpy="0 0 0" />
     <parent
-      link="camera_bottom_screw_frame" />
-    <child
-      link="camera_IR2_frame" />
-    <axis
-      xyz="0 0 0" />
-  </joint>
-  <link
-    name="camera_IR2_optical_frame">
+      link="camera_depth_frame" />
+    <child
+      link="camera_right_ir_frame" />
+    <axis
+      xyz="0 0 0" />
+  </joint>
+  <link
+    name="camera_right_ir_optical_frame">
     <inertial>
       <origin
@@ -192,5 +192,5 @@
   </link>
   <joint
-    name="camera_IR2_optical_frame"
+    name="camera_right_ir_optical_frame"
     type="fixed">
     <origin
@@ -198,12 +198,12 @@
       rpy="-1.5708 0 -1.5708" />
     <parent
-      link="camera_IR2_frame" />
-    <child
-      link="camera_IR2_optical_frame" />
-    <axis
-      xyz="0 0 0" />
-  </joint>
-  <link
-    name="camera_IR1_frame">
+      link="camera_right_ir_frame" />
+    <child
+      link="camera_right_ir_optical_frame" />
+    <axis
+      xyz="0 0 0" />
+  </joint>
+  <link
+    name="camera_left_ir_frame">
     <inertial>
       <origin
@@ -245,18 +245,18 @@
   </link>
   <joint
-    name="camera_IR1_frame"
-    type="fixed">
-    <origin
-      xyz="0.01033 0.05 0.0145"
+    name="camera_left_ir_frame"
+    type="fixed">
+    <origin
+      xyz="0 0 0"
       rpy="0 0 0" />
     <parent
-      link="camera_bottom_screw_frame" />
-    <child
-      link="camera_IR1_frame" />
-    <axis
-      xyz="0 0 0" />
-  </joint>
-  <link
-    name="camera_IR1_optical_frame">
+      link="camera_depth_frame" />
+    <child
+      link="camera_left_ir_frame" />
+    <axis
+      xyz="0 0 0" />
+  </joint>
+  <link
+    name="camera_left_ir_optical_frame">
     <inertial>
       <origin
@@ -298,5 +298,5 @@
   </link>
   <joint
-    name="camera_IR1_optical_frame"
+    name="camera_left_ir_optical_frame"
     type="fixed">
     <origin
@@ -304,7 +304,7 @@
       rpy="-1.5708 0 -1.5708" />
     <parent
-      link="camera_IR1_frame" />
-    <child
-      link="camera_IR1_optical_frame" />
+      link="camera_left_ir_frame" />
+    <child
+      link="camera_left_ir_optical_frame" />
     <axis
       xyz="0 0 0" />
@@ -354,8 +354,8 @@
     type="fixed">
     <origin
-      xyz="0.010330000039789 0.025 0.0145"
+      xyz="3.9789e-11 -0.025 0"
       rpy="0 0 0" />
     <parent
-      link="camera_bottom_screw_frame" />
+      link="camera_depth_frame" />
     <child
       link="camera_color_frame" />
@@ -364,5 +364,5 @@
   </joint>
   <link
-    name="camera_rgb_optical_frame">
+    name="camera_color_optical_frame">
     <inertial>
       <origin
@@ -404,5 +404,5 @@
   </link>
   <joint
-    name="camera_rgb_optical_frame"
+    name="camera_color_optical_frame"
     type="fixed">
     <origin
@@ -412,5 +412,5 @@
       link="camera_color_frame" />
     <child
-      link="camera_rgb_optical_frame" />
+      link="camera_color_optical_frame" />
     <axis
       xyz="0 0 0" />
@@ -460,8 +460,8 @@
     type="fixed">
     <origin
-      xyz="-0.00473999996021007 0.034841019999999 0.017079659999999"
+      xyz="-0.01507 -0.015159 0.0025797"
       rpy="0 0 0" />
     <parent
-      link="camera_bottom_screw_frame" />
+      link="camera_depth_frame" />
     <child
       link="camera_imu_frame" />
@@ -513,8 +513,8 @@
     type="fixed">
     <origin
-      xyz="0.010330000039789 0.05 0.0145"
+      xyz="0 0 0"
       rpy="0 0 0" />
     <parent
-      link="camera_bottom_screw_frame" />
+      link="camera_link" />
     <child
       link="camera_depth_frame" />

File: urdf/gemini335L_336L.urdf.xacro (robot description, xacro)
@@ -23,5 +23,5 @@
     <visual>
       <origin
-        xyz="0 0 0"
+        xyz="-0.011715 -0.0475 -0.014311"
         rpy="0 0 0" />
       <geometry>
@@ -89,5 +89,5 @@
     type="fixed">
     <origin
-      xyz="0 0 0"
+      xyz="-0.011715 -0.0475 -0.014311"
       rpy="0 0 0" />
     <parent
@@ -142,8 +142,8 @@
     type="fixed">
     <origin
-      xyz="-0.002535 0.039634 0.013243"
+      xyz="-0.01425 -0.007866 -0.001068"
       rpy="0 0 0" />
     <parent
-      link="camera_color_screw_frame" />
+      link="camera_depth_frame" />
     <child
       link="camera_IMU_frame" />
@@ -195,8 +195,8 @@
     type="fixed">
     <origin
-      xyz="0.011715 0.0475 0.014311"
+      xyz="0 0 0"
       rpy="0 0 0" />
     <parent
-      link="camera_color_screw_frame" />
+      link="camera_link" />
     <child
       link="camera_depth_frame" />
@@ -205,5 +205,5 @@
   </joint>
   <link
-    name="camera_infra1_frame">
+    name="camera_left_ir_frame">
     <inertial>
       <origin
@@ -245,18 +245,18 @@
   </link>
   <joint
-    name="camera_infra1_frame"
-    type="fixed">
-    <origin
-      xyz="0.011715 0.0475 0.014311"
+    name="camera_left_ir_frame"
+    type="fixed">
+    <origin
+      xyz="0 0 0"
       rpy="0 0 0" />
     <parent
-      link="camera_color_screw_frame" />
-    <child
-      link="camera_infra1_frame" />
-    <axis
-      xyz="0 0 0" />
-  </joint>
-  <link
-    name="camera_infra1_optical_frame">
+      link="camera_depth_frame" />
+    <child
+      link="camera_left_ir_frame" />
+    <axis
+      xyz="0 0 0" />
+  </joint>
+  <link
+    name="camera_left_ir_optical_frame">
     <inertial>
       <origin
@@ -298,5 +298,5 @@
   </link>
   <joint
-    name="camera_infra1_optical_frame"
+    name="camera_left_ir_optical_frame"
     type="fixed">
     <origin
@@ -304,12 +304,12 @@
       rpy="-1.5708 0 -1.5708" />
     <parent
-      link="camera_infra1_frame" />
-    <child
-      link="camera_infra1_optical_frame" />
-    <axis
-      xyz="0 0 0" />
-  </joint>
-  <link
-    name="camera_infra2_frame">
+      link="camera_left_ir_frame" />
+    <child
+      link="camera_left_ir_optical_frame" />
+    <axis
+      xyz="0 0 0" />
+  </joint>
+  <link
+    name="camera_right_ir_frame">
     <inertial>
       <origin
@@ -351,18 +351,18 @@
   </link>
   <joint
-    name="camera_infra2_frame"
-    type="fixed">
-    <origin
-      xyz="0.011715 -0.0475 0.014311"
+    name="camera_right_ir_frame"
+    type="fixed">
+    <origin
+      xyz="0 -0.095 0"
       rpy="0 0 0" />
     <parent
-      link="camera_color_screw_frame" />
-    <child
-      link="camera_infra2_frame" />
-    <axis
-      xyz="0 0 0" />
-  </joint>
-  <link
-    name="camera_infra2_optical_frame">
+      link="camera_depth_frame" />
+    <child
+      link="camera_right_ir_frame" />
+    <axis
+      xyz="0 0 0" />
+  </joint>
+  <link
+    name="camera_right_ir_optical_frame">
     <inertial>
       <origin
@@ -404,5 +404,5 @@
   </link>
   <joint
-    name="camera_infra2_optical_frame"
+    name="camera_right_ir_optical_frame"
     type="fixed">
     <origin
@@ -410,7 +410,7 @@
       rpy="-1.5708 0 -1.5708" />
     <parent
-      link="camera_infra2_frame" />
-    <child
-      link="camera_infra2_optical_frame" />
+      link="camera_right_ir_frame" />
+    <child
+      link="camera_right_ir_optical_frame" />
     <axis
       xyz="0 0 0" />
@@ -460,8 +460,8 @@
     type="fixed">
     <origin
-      xyz="0.011715 0.02375 0.014311"
+      xyz="0 -0.02375 0"
       rpy="0.0010157 0 0" />
     <parent
-      link="camera_color_screw_frame" />
+      link="camera_depth_frame" />
     <child
       link="camera_color_frame" />

File: urdf/gemini_335_336.urdf.xacro (robot description, xacro)
@@ -4,5 +4,5 @@
      Commit Version: 1.6.0-4-g7f85cfe  Build Version: 1.6.7995.38578
      For more information, please see http://wiki.ros.org/sw_urdf_exporter -->
-<robot xmlns:xacro="http://ros.org/wiki/xacro" name="gemini335_336">
+<robot xmlns:xacro="http://ros.org/wiki/xacro" name="gemini_335_336">
     <xacro:property name="mesh_path" value="package://orbbec_camera/meshes/gemini335_336/" />
     <link name="camera_link">
@@ -15,5 +15,5 @@
         </inertial>
         <visual>
-            <origin xyz="0 0 0" rpy="0 0 0" />
+            <origin xyz="-0.01587 -0.025 -0.0125" rpy="0 0 0" />
             <geometry>
                 <mesh filename="${mesh_path}camera_link.STL" />
@@ -55,5 +55,5 @@
     </link>
     <joint name="camera_bottom_screw_frame_joint" type="fixed">
-        <origin xyz="0 0 0" rpy="0 0 0" />
+        <origin xyz="-0.01587 -0.025 -0.0125" rpy="0 0 0" />
         <parent link="camera_link" />
         <child link="camera_bottom_screw_frame" />
@@ -86,6 +86,6 @@
     </link>
     <joint name="camera_left_ir_joint" type="fixed">
-        <origin xyz="0.01587 -0.025 0.0125" rpy="0 0 0" />
-        <parent link="camera_bottom_screw_frame" />
+        <origin xyz="0 0 0" rpy="0 0 0" />
+        <parent link="camera_depth_frame" />
         <child link="camera_left_ir_frame" />
         <axis xyz="0 0 0" />
@@ -116,6 +116,6 @@
     </link>
     <joint name="camera_left_ir_optical_joint" type="fixed">
-        <origin xyz="0.01587 -0.025 0.0125" rpy="-1.5707963267949 0 -1.5707963267949" />
-        <parent link="camera_bottom_screw_frame" />
+        <origin xyz="0 0 0" rpy="-1.5707963267949 0 -1.5707963267949" />
+        <parent link="camera_left_ir_frame" />
         <child link="camera_left_ir_optical_frame" />
         <axis xyz="0 0 0" />
@@ -147,6 +147,6 @@
     </link>
     <joint name="camera_right_ir_joint" type="fixed">
-        <origin xyz="0.01587 0.025 0.0125" rpy="0 0 0" />
-        <parent link="camera_bottom_screw_frame" />
+        <origin xyz="0 -0.05 0" rpy="0 0 0" />
+        <parent link="camera_depth_frame" />
         <child link="camera_right_ir_frame" />
         <axis xyz="0 0 0" />
@@ -177,6 +177,6 @@
     </link>
     <joint name="camera_right_ir_optical_joint" type="fixed">
-        <origin xyz="0.01587 0.025 0.0125" rpy="-1.5707963267949 0 -1.5707963267949" />
-        <parent link="camera_bottom_screw_frame" />
+        <origin xyz="0 0 0" rpy="-1.5707963267949 0 -1.5707963267949" />
+        <parent link="camera_right_ir_frame" />
         <child link="camera_right_ir_optical_frame" />
         <axis xyz="0 0 0" />
@@ -208,6 +208,6 @@
     </link>
     <joint name="camera_color_joint" type="fixed">
-        <origin xyz="0.017533 0.010995 0.012505" rpy="0 0 0" />
-        <parent link="camera_bottom_screw_frame" />
+        <origin xyz="0.001663 -0.014005 0.000005" rpy="0 0 0" />
+        <parent link="camera_depth_frame" />
         <child link="camera_color_frame" />
         <axis xyz="0 0 0" />
@@ -239,6 +239,6 @@
     </link>
     <joint name="camera_color_optical_joint" type="fixed">
-        <origin xyz="0.017533 0.010995 0.012505" rpy="-1.5707963267949 0 -1.5707963267949" />
-        <parent link="camera_bottom_screw_frame" />
+        <origin xyz="0 0 0" rpy="-1.5707963267949 0 -1.5707963267949" />
+        <parent link="camera_color_frame" />
         <child link="camera_color_optical_frame" />
         <axis xyz="0 0 0" />
@@ -270,6 +270,6 @@
     </link>
     <joint name="camera_depth_joint" type="fixed">
-        <origin xyz="0.01587 -0.025 0.0125" rpy="0 0 0" />
-        <parent link="camera_bottom_screw_frame" />
+        <origin xyz="0 0 0" rpy="0 0 0" />
+        <parent link="camera_link" />
         <child link="camera_depth_frame" />
         <axis xyz="0 0 0" />
@@ -299,6 +299,6 @@
     </link>
     <joint name="camera_depth_optical_joint" type="fixed">
-        <origin xyz="0.01587 -0.025 0.0125" rpy="-1.5707963267949 0 -1.5707963267949" />
-        <parent link="camera_bottom_screw_frame" />
+        <origin xyz="0 0 0" rpy="-1.5707963267949 0 -1.5707963267949" />
+        <parent link="camera_depth_frame" />
         <child link="camera_depth_optical_frame" />
         <axis xyz="0 0 0" />

File: urdf/test_astra2.urdf.xacro (robot description, xacro)
@@ -3,6 +3,6 @@
      Commit Version: 1.6.0-4-g7f85cfe  Build Version: 1.6.7995.38578
      For more information, please see http://wiki.ros.org/sw_urdf_exporter -->
-<robot name="gemini335" xmlns:xacro="http://ros.org/wiki/xacro">
-    <xacro:include filename="gemini335_336.urdf.xacro"/>
+<robot name="astra2" xmlns:xacro="http://ros.org/wiki/xacro">
+    <xacro:include filename="astra2.urdf.xacro"/>
     <!-- Define a virtual root link -->
   <link name="base_link"/>
@@ -11,5 +11,5 @@
     <parent link="base_link"/>
     <child link="camera_link"/>
-    <origin xyz="0 0 0" rpy="0 0 0"/>
+    <origin xyz="0.012323996052145958 0.03750000149011612 0.028150320053100586" rpy="0 0 0"/>
   </joint>
 </robot>

File: urdf/test_gemini2.urdf.xacro (robot description, xacro)
@@ -3,6 +3,6 @@
      Commit Version: 1.6.0-4-g7f85cfe  Build Version: 1.6.7995.38578
      For more information, please see http://wiki.ros.org/sw_urdf_exporter -->
-<robot name="astra2" xmlns:xacro="http://ros.org/wiki/xacro">
-    <xacro:include filename="astra2.urdf.xarco"/>
+<robot name="gemini2" xmlns:xacro="http://ros.org/wiki/xacro">
+    <xacro:include filename="gemini2.urdf.xacro"/>
     <!-- Define a virtual root link -->
   <link name="base_link"/>
@@ -11,5 +11,5 @@
     <parent link="base_link"/>
     <child link="camera_link"/>
-    <origin xyz="0 0 0" rpy="0 0 0"/>
+    <origin xyz="0.01491 0.025 0.0125" rpy="0 0 0"/>
   </joint>
 </robot>

File: urdf/test_gemini2L.urdf.xacro (robot description, xacro)
@@ -3,6 +3,6 @@
      Commit Version: 1.6.0-4-g7f85cfe  Build Version: 1.6.7995.38578
      For more information, please see http://wiki.ros.org/sw_urdf_exporter -->
-<robot name="gemini336" xmlns:xacro="http://ros.org/wiki/xacro">
-    <xacro:include filename="gemini335_336.urdf.xacro"/>
+<robot name="gemini2L" xmlns:xacro="http://ros.org/wiki/xacro">
+    <xacro:include filename="gemini2L.urdf.xacro"/>
     <!-- Define a virtual root link -->
   <link name="base_link"/>
@@ -11,5 +11,5 @@
     <parent link="base_link"/>
     <child link="camera_link"/>
-    <origin xyz="0 0 0" rpy="0 0 0"/>
+    <origin xyz="0.01033 0.05 0.0145" rpy="0 0 0"/>
   </joint>
 </robot>

File: urdf/test_gemini336L.urdf.xacro (robot description, xacro)
@@ -3,6 +3,6 @@
      Commit Version: 1.6.0-4-g7f85cfe  Build Version: 1.6.7995.38578
      For more information, please see http://wiki.ros.org/sw_urdf_exporter -->
-<robot name="gemini2" xmlns:xacro="http://ros.org/wiki/xacro">
-    <xacro:include filename="gemini2.urdf.xarco"/>
+<robot name="gemini336L" xmlns:xacro="http://ros.org/wiki/xacro">
+    <xacro:include filename="gemini335L_336L.urdf.xacro"/>
     <!-- Define a virtual root link -->
   <link name="base_link"/>
@@ -11,5 +11,5 @@
     <parent link="base_link"/>
     <child link="camera_link"/>
-    <origin xyz="0 0 0" rpy="0 0 0"/>
+    <origin xyz="0.011715 0.0475 0.014311" rpy="0 0 0"/>
   </joint>
 </robot>

File: urdf/test_gemini_335.urdf.xacro (robot description, xacro)
@@ -3,6 +3,6 @@
      Commit Version: 1.6.0-4-g7f85cfe  Build Version: 1.6.7995.38578
      For more information, please see http://wiki.ros.org/sw_urdf_exporter -->
-<robot name="gemini2L" xmlns:xacro="http://ros.org/wiki/xacro">
-    <xacro:include filename="gemini2L.urdf.xarco"/>
+<robot name="gemini_335" xmlns:xacro="http://ros.org/wiki/xacro">
+    <xacro:include filename="gemini_335_336.urdf.xacro"/>
     <!-- Define a virtual root link -->
   <link name="base_link"/>
@@ -11,5 +11,5 @@
     <parent link="base_link"/>
     <child link="camera_link"/>
-    <origin xyz="0 0 0" rpy="0 0 0"/>
+    <origin xyz="0.01587 0.025 0.0125" rpy="0 0 0"/>
   </joint>
 </robot>
