Commit message: fix: update collision origin positions in URDF files

File: urdf/astra2.urdf.xacro (robot description, xacro)
@@ -37,5 +37,5 @@
     <collision>
       <origin
-        xyz="0 0 0"
+        xyz="-0.012323995999904 -0.0374999999985815 -0.0281503197112"
         rpy="0 0 0" />
       <geometry>

File: urdf/gemini2.urdf.xacro (robot description, xacro)
@@ -37,5 +37,5 @@
     <collision>
       <origin
-        xyz="0 0 0"
+        xyz="-0.01491 -0.025 -0.0125"
         rpy="0 0 0" />
       <geometry>

File: urdf/gemini2L.urdf.xacro (robot description, xacro)
@@ -37,5 +37,5 @@
     <collision>
       <origin
-        xyz="0 0 0"
+        xyz="-0.01033 -0.05 -0.0145"
         rpy="0 0 0" />
       <geometry>

File: urdf/gemini335L_336L.urdf.xacro (robot description, xacro)
@@ -37,5 +37,5 @@
     <collision>
       <origin
-        xyz="0 0 0"
+        xyz="-0.011715 -0.0475 -0.014311"
         rpy="0 0 0" />
       <geometry>

File: urdf/gemini335Le.urdf.xacro (robot description, xacro)
@@ -38,5 +38,5 @@
     <collision>
       <origin
-        xyz="0 0 0"
+        xyz="-0.034005 -0.0475 -0.014048"
         rpy="0 0 0" />
       <geometry>

File: urdf/gemini335Lg.urdf.xacro (robot description, xacro)
@@ -38,5 +38,5 @@
     <collision>
       <origin
-        xyz="0 0 0"
+        xyz="-0.0117149999999995 -0.0475 -0.0143111800025738"
         rpy="0 0 0" />
       <geometry>

File: urdf/gemini_335_336.urdf.xacro (robot description, xacro)
@@ -24,5 +24,5 @@
         </visual>
         <collision>
-            <origin xyz="0 0 0" rpy="0 0 0" />
+            <origin xyz="-0.01587 -0.025 -0.0125" rpy="0 0 0" />
             <geometry>
                 <mesh filename="${mesh_path}camera_link.STL" />
