Commit message: Rename Gemini URDF files consistently

File: urdf/gemini_335_L_336_L.urdf.xacro (robot description, xacro)
@@ -3,25 +3,25 @@
      Commit Version: 1.6.0-4-g7f85cfe  Build Version: 1.6.7995.38578
      For more information, please see http://wiki.ros.org/sw_urdf_exporter -->
-<robot xmlns:xacro="http://ros.org/wiki/xacro" name="gemini2l">
-    <xacro:property name="mesh_path" value="package://orbbec_camera/meshes/gemini2l/" />
+<robot xmlns:xacro="http://ros.org/wiki/xacro" name="gemini_335_L_336_L">
+    <xacro:property name="mesh_path" value="package://orbbec_camera/meshes/gemini335L_336L/" />
   <link
     name="camera_link">
     <inertial>
       <origin
-        xyz="-0.0011764 -0.00036824 0.013857"
-        rpy="0 0 0" />
-      <mass
-        value="0.0063118" />
-      <inertia
-        ixx="6.2823E-06"
-        ixy="-1.425E-09"
-        ixz="4.3925E-09"
-        iyy="3.0429E-07"
-        iyz="2.3803E-08"
-        izz="6.0224E-06" />
-    </inertial>
-    <visual>
-      <origin
-        xyz="-0.01033 -0.05 -0.0145"
+        xyz="0.00287577972418718 0.000617475958990782 0.0141094270811986"
+        rpy="0 0 0" />
+      <mass
+        value="0.0330710167577971" />
+      <inertia
+        ixx="4.44764516625696E-05"
+        ixy="5.53948591538607E-08"
+        ixz="-2.79060738018455E-08"
+        iyy="3.07720636867613E-06"
+        iyz="1.65209163393457E-07"
+        izz="4.23385079682874E-05" />
+    </inertial>
+    <visual>
+      <origin
+        xyz="-0.011715 -0.0475 -0.014311"
         rpy="0 0 0" />
       <geometry>
@@ -32,10 +32,10 @@
         name="">
         <color
-          rgba="0.79216 0.81961 0.93333 1" />
-      </material>
-    </visual>
-    <collision>
-      <origin
-        xyz="-0.01033 -0.05 -0.0145"
+          rgba="0.792156862745098 0.819607843137255 0.933333333333333 1" />
+      </material>
+    </visual>
+    <collision>
+      <origin
+        xyz="-0.011715 -0.0475 -0.014311"
         rpy="0 0 0" />
       <geometry>
@@ -46,151 +46,257 @@
   </link>
   <link
-    name="camera_bottom_screw_frame">
-    <inertial>
-      <origin
-        xyz="0.0029372 -0.00037745 0.014561"
-        rpy="0 0 0" />
-      <mass
-        value="0.037165" />
-      <inertia
-        ixx="4.9388E-05"
-        ixy="-4.4007E-08"
-        ixz="-6.3785E-09"
-        iyy="3.6527E-06"
-        iyz="6.164E-08"
-        izz="4.6538E-05" />
-    </inertial>
-    <visual>
-      <origin
-        xyz="0 0 0"
-        rpy="0 0 0" />
-      <geometry>
-        <mesh
-          filename="${mesh_path}camera_bottom_screw_frame.STL" />
-      </geometry>
-      <material
-        name="">
-        <color
-          rgba="0.79216 0.81961 0.93333 1" />
-      </material>
-    </visual>
-    <collision>
-      <origin
-        xyz="0 0 0"
-        rpy="0 0 0" />
-      <geometry>
-        <mesh
-          filename="${mesh_path}camera_bottom_screw_frame.STL" />
-      </geometry>
-    </collision>
-  </link>
-  <joint
-    name="camera_bottom_screw_joint"
-    type="fixed">
-    <origin
-      xyz="-0.01033 -0.05 -0.0145"
+    name="camera_color_screw_frame">
+    <inertial>
+      <origin
+        xyz="-0.000565327084882765 -0.000754794567604389 0.0132965378040367"
+        rpy="0 0 0" />
+      <mass
+        value="0.00682237197281727" />
+      <inertia
+        ixx="6.29665283187838E-06"
+        ixy="-5.56290557545124E-09"
+        ixz="-4.00728156039594E-09"
+        iyy="3.51296306719609E-07"
+        iyz="1.01025992411894E-07"
+        izz="5.98951376451163E-06" />
+    </inertial>
+    <visual>
+      <origin
+        xyz="0 0 0"
+        rpy="0 0 0" />
+      <geometry>
+        <mesh
+          filename="${mesh_path}camera_color_screw_frame.STL" />
+      </geometry>
+      <material
+        name="">
+        <color
+          rgba="0.792156862745098 0.819607843137255 0.933333333333333 1" />
+      </material>
+    </visual>
+    <collision>
+      <origin
+        xyz="0 0 0"
+        rpy="0 0 0" />
+      <geometry>
+        <mesh
+          filename="${mesh_path}camera_color_screw_frame.STL" />
+      </geometry>
+    </collision>
+  </link>
+  <joint
+    name="camera_color_screw_joint"
+    type="fixed">
+    <origin
+      xyz="-0.011715 -0.0475 -0.014311"
       rpy="0 0 0" />
     <parent
       link="camera_link" />
     <child
-      link="camera_bottom_screw_frame" />
-    <axis
-      xyz="0 0 0" />
-  </joint>
-  <link
-    name="camera_right_ir_frame">
-    <inertial>
-      <origin
-        xyz="0.00133699020857289 -3.04478174825706E-08 3.7713891998328E-08"
-        rpy="0 0 0" />
-      <mass
-        value="0.000234825886837936" />
-      <inertia
-        ixx="2.7973722771565E-09"
-        ixy="4.86630909822049E-16"
-        ixz="-6.02474175028887E-16"
-        iyy="1.60708521944039E-09"
-        iyz="2.50471029328346E-14"
-        izz="1.60707326572337E-09" />
-    </inertial>
-    <visual>
-      <origin
-        xyz="0 0 0"
-        rpy="0 0 0" />
-      <geometry>
-        <mesh
-          filename="${mesh_path}camera_IR2_frame.STL" />
-      </geometry>
-      <material
-        name="">
-        <color
-          rgba="0.501960784313725 0.250980392156863 0.250980392156863 1" />
-      </material>
-    </visual>
-    <collision>
-      <origin
-        xyz="0 0 0"
-        rpy="0 0 0" />
-      <geometry>
-        <mesh
-          filename="${mesh_path}camera_IR2_frame.STL" />
-      </geometry>
-    </collision>
-  </link>
-  <joint
-    name="camera_right_ir_joint"
-    type="fixed">
-    <origin
-      xyz="0 -0.1 0"
+      link="camera_color_screw_frame" />
+    <axis
+      xyz="0 0 0" />
+  </joint>
+  <link
+    name="camera_IMU_frame">
+    <inertial>
+      <origin
+        xyz="-0.000484999999999999 0 0"
+        rpy="0 0 0" />
+      <mass
+        value="1.1218632E-05" />
+      <inertia
+        ixx="2.18587565431999E-11"
+        ixy="0"
+        ixz="-3.24383195391647E-28"
+        iyy="1.0215031879E-11"
+        iyz="-3.36058814408671E-29"
+        izz="1.34029931389999E-11" />
+    </inertial>
+    <visual>
+      <origin
+        xyz="0 0 0"
+        rpy="0 0 0" />
+      <geometry>
+        <mesh
+          filename="${mesh_path}camera_IMU_frame.STL" />
+      </geometry>
+      <material
+        name="">
+        <color
+          rgba="0.792156862745098 0.819607843137255 0.933333333333333 1" />
+      </material>
+    </visual>
+    <collision>
+      <origin
+        xyz="0 0 0"
+        rpy="0 0 0" />
+      <geometry>
+        <mesh
+          filename="${mesh_path}camera_IMU_frame.STL" />
+      </geometry>
+    </collision>
+  </link>
+  <joint
+    name="camera_IMU_joint"
+    type="fixed">
+    <origin
+      xyz="-0.01425 -0.007866 -0.001068"
       rpy="0 0 0" />
     <parent
       link="camera_depth_frame" />
     <child
-      link="camera_right_ir_frame" />
-    <axis
-      xyz="0 0 0" />
-  </joint>
-  <link
-    name="camera_right_ir_optical_frame">
-    <inertial>
-      <origin
-        xyz="3.04478174825706E-08 -3.77138919982661E-08 0.00133699020857289"
-        rpy="0 0 0" />
-      <mass
-        value="0.000234825886837936" />
-      <inertia
-        ixx="1.60708521944039E-09"
-        ixy="2.50471029328366E-14"
-        ixz="-4.86630909830569E-16"
-        iyy="1.60707326572337E-09"
-        iyz="6.02474175031465E-16"
-        izz="2.7973722771565E-09" />
-    </inertial>
-    <visual>
-      <origin
-        xyz="0 0 0"
-        rpy="0 0 0" />
-      <geometry>
-        <mesh
-          filename="${mesh_path}camera_IR2_optical_frame.STL" />
-      </geometry>
-      <material
-        name="">
-        <color
-          rgba="0.501960784313725 0.250980392156863 0.250980392156863 1" />
-      </material>
-    </visual>
-    <collision>
-      <origin
-        xyz="0 0 0"
-        rpy="0 0 0" />
-      <geometry>
-        <mesh
-          filename="${mesh_path}camera_IR2_optical_frame.STL" />
-      </geometry>
-    </collision>
-  </link>
-  <joint
-    name="camera_right_ir_optical_joint"
+      link="camera_IMU_frame" />
+    <axis
+      xyz="0 0 0" />
+  </joint>
+  <link
+    name="camera_depth_frame">
+    <inertial>
+      <origin
+        xyz="-0.00158020638644197 -1.72113892998871E-08 -1.52265896501485E-07"
+        rpy="0 0 0" />
+      <mass
+        value="0.00045316775745635" />
+      <inertia
+        ixx="4.34107394943177E-09"
+        ixy="-3.70457372455813E-13"
+        ixz="-1.46474854133768E-13"
+        iyy="4.84011101176503E-09"
+        iyz="2.21976196909378E-14"
+        izz="4.84043649602512E-09" />
+    </inertial>
+    <visual>
+      <origin
+        xyz="0 0 0"
+        rpy="0 0 0" />
+      <geometry>
+        <mesh
+          filename="${mesh_path}camera_depth_frame.STL" />
+      </geometry>
+      <material
+        name="">
+        <color
+          rgba="0.792156862745098 0.819607843137255 0.933333333333333 1" />
+      </material>
+    </visual>
+    <collision>
+      <origin
+        xyz="0 0 0"
+        rpy="0 0 0" />
+      <geometry>
+        <mesh
+          filename="${mesh_path}camera_depth_frame.STL" />
+      </geometry>
+    </collision>
+  </link>
+  <joint
+    name="camera_depth_joint"
+    type="fixed">
+    <origin
+      xyz="0 0 0"
+      rpy="0 0 0" />
+    <parent
+      link="camera_link" />
+    <child
+      link="camera_depth_frame" />
+    <axis
+      xyz="0 0 0" />
+  </joint>
+  <link
+    name="camera_left_ir_frame">
+    <inertial>
+      <origin
+        xyz="-0.00158020638644197 -1.72113892998871E-08 -1.52265896501463E-07"
+        rpy="0 0 0" />
+      <mass
+        value="0.00045316775745635" />
+      <inertia
+        ixx="4.34107394943177E-09"
+        ixy="-3.70457372455807E-13"
+        ixz="-1.464748541338E-13"
+        iyy="4.84011101176503E-09"
+        iyz="2.21976196909559E-14"
+        izz="4.84043649602512E-09" />
+    </inertial>
+    <visual>
+      <origin
+        xyz="0 0 0"
+        rpy="0 0 0" />
+      <geometry>
+        <mesh
+          filename="${mesh_path}camera_infra1_frame.STL" />
+      </geometry>
+      <material
+        name="">
+        <color
+          rgba="0.792156862745098 0.819607843137255 0.933333333333333 1" />
+      </material>
+    </visual>
+    <collision>
+      <origin
+        xyz="0 0 0"
+        rpy="0 0 0" />
+      <geometry>
+        <mesh
+          filename="${mesh_path}camera_infra1_frame.STL" />
+      </geometry>
+    </collision>
+  </link>
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
File: urdf/gemini_335_Le.urdf.xacro (robot description, xacro)
@@ -4,5 +4,5 @@
      Commit Version: 1.6.0-4-g7f85cfe  Build Version: 1.6.7995.38578
      For more information, please see http://wiki.ros.org/sw_urdf_exporter -->
-<robot xmlns:xacro="http://ros.org/wiki/xacro" name="gemini335Le">
+<robot xmlns:xacro="http://ros.org/wiki/xacro" name="gemini_335_Le">
     <xacro:property name="mesh_path" value="package://orbbec_camera/meshes/gemini335Le/" />
    <link

File: urdf/gemini_335_Lg.urdf.xacro (robot description, xacro)
@@ -4,5 +4,5 @@
      Commit Version: 1.6.0-4-g7f85cfe  Build Version: 1.6.7995.38578
      For more information, please see http://wiki.ros.org/sw_urdf_exporter -->
-<robot xmlns:xacro="http://ros.org/wiki/xacro" name="gemini335_336Lg">
+<robot xmlns:xacro="http://ros.org/wiki/xacro" name="gemini_335_Lg">
     <xacro:property name="mesh_path" value="package://orbbec_camera/meshes/gemini335Lg/" />
     <link
